File: eagle/v4/schematics.brd (EAGLE design)
At the start: 49.5 x 27.6 mm, 38 parts, among them J1 TYPE-C-31-M-12, T1 MMBT2222A, U1 SN74LVC2G14

Commit message: HW4.1
Parts:
- removed TELEINFO: (no value), con-wago-500:W237-102
- added TIC1, TIC2: WIREPAD2,15/1,0, wirepad:2,15/1,0
- RESET, S1: value MICROSWITCH -> TS-1088-AR02016; device Nicolas:MICROSWITCH -> TS-1088-AR02016:SW_TS-1088-AR02016
- moved D1 3.33 mm to (7.57, 6.07), turned to 90 degrees
- moved S1 1.27 mm to (39.4, 11.4)
- moved RESET 0.25 mm to (39.4, 3.81)
Connections:
- net N$7: now also TIC1.1; no longer TELEINFO.1
- net N$8: now also TIC2.1; no longer TELEINFO.2
Routing:
- net N$12: track 3.26 -> 6.74 mm
- net N$8: track 19.2 -> 16.1 mm
- net N$10: track 8.25 -> 10.4 mm
- net N$4: track 42.7 -> 44.8 mm
- net N$7: track 10.8 -> 10.1 mm
Other:
- board text added: "S1"
- board text added: "TeleInfoKit v4.1"
- board text removed: "TeleInfoKit v4"
