File: eagle/v4/schematics.sch (EAGLE design)
At the start: 38 parts, among them J1 TYPE-C-31-M-12, T1 MMBT2222A, U1 SN74LVC2G14

Commit message: HW4.1
Parts:
- removed TELEINFO: (no value), con-wago-500:W237-102
- added TIC1, TIC2: WIREPAD2,15/1,0, wirepad:WIREPAD2,15/1,0
- ESP: LCSC_PART (none) -> C2935984
- OK1: LCSC_PART (none) -> C479718
- OLED: LCSC_PART (none) -> C2718488
- RESET, S1: value MICROSWITCH -> TS-1088-AR02016; device Nicolas:MICROSWITCH -> TS-1088-AR02016:TS-1088-AR02016; LCSC_PART (none) -> C720477
Connections:
- net N$7: now also TIC1.P; no longer TELEINFO-1.KL
- net N$8: now also TIC2.P; no longer TELEINFO-2.KL
Other:
- note added: "Teleinfokit v4.1"
- note removed: "Teleinfokit v4"
- moved on the sheet: RESET, S1
