File: eagle/v5/schematics.sch (EAGLE design)
At the start: 25 parts, among them T1 MMBT2222A, U1 SN74LVC2G14

Commit message: V5 update
Parts:
- removed C2, C4: 1uF, rcl:C-EUC0805
- removed C3: 4.7uF, rcl:C-EUC0805
- removed C5: 0.1uF, rcl:C-EUC0402K
- removed POWER: (no value), pinhead:PINHD-1X3
- removed R6: 300, rcl:R-EU_R0805
- added 5V: (no value), adafruit:PINHD-1X1
- added JP3: (no value), adafruit:PINHD-1X3
- added R3: 1k, rcl:R-EU_R0805
- C1: value 4.7uF -> 0.1uF; device rcl:C-EUC0805 -> rcl:C-EUC0402K; LCSC_PART C1779 -> C1525
- R4: value 1k -> 10k
- R5: value 10k -> 300; LCSC_PART C17414 -> C17617
Connections:
- net +3V3: now also C1.1, R5.1; no longer C3.1, C4.1, C5.1, POWER.1, R6.1
- net +5V: now also 5V.1; no longer C1.1, C2.1, POWER.2
- net GND: now also JP3.1; no longer C2.2, C3.2, C4.2, C5.2, POWER.3
- net N$13: now also R4.2; no longer R5.2
- net N$15: now also R3.1; no longer R4.1
- net N$3: now also R5.2; no longer R6.2
- net N$5: now also R4.1; no longer R5.1
- net RXD: now also JP3.3, R3.2; no longer R4.2
- net TXD: now also JP3.2
Other:
- moved on the sheet: C1, R4, R5

Commit message: V5 update
Connections:
- net N$10 renamed IO5
- net N$14 renamed IO6
- net N$16 renamed IO7
- net N$17 renamed IO10
- net N$18 renamed IO4
- net N$19 renamed IO3
- net N$2 renamed SDA
- net N$20 renamed IO2
- net N$21 renamed IO1
- net N$6 renamed SCL
Changed lines of the file:
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@@
 </segment>
 </net>
-<net name="N$2" class="0">
+<net name="SDA" class="0">
 <segment>
 <pinref part="OLED" gate="G$1" pin="SDA"/>
@@
 <pinref part="U$1" gate="G$1" pin="G8"/>
 <wire x1="104.14" y1="60.96" x2="129.54" y2="60.96" width="0.1524" layer="91"/>
-</segment>
-</net>
-<net name="N$6" class="0">
+<label x="124.46" y="60.96" size="1.778" layer="95" rot="R270" xref="yes"/>
+</segment>
+</net>
+<net name="SCL" class="0">
 <segment>
 <pinref part="OLED" gate="G$1" pin="SCL"/>
@@
 <pinref part="U$1" gate="G$1" pin="G9"/>
 <wire x1="104.14" y1="63.5" x2="132.08" y2="63.5" width="0.1524" layer="91"/>
+<label x="132.08" y="60.96" size="1.778" layer="95" xref="yes"/>
 </segment>
 </net>
@@
 </segment>
 </net>
-<net name="N$10" class="0">
+<net name="IO5" class="0">
 <segment>
 <pinref part="JP1" gate="A" pin="5"/>
@@
 </segment>
 </net>
-<net name="N$14" class="0">
+<net name="IO6" class="0">
 <segment>
 <pinref part="U$1" gate="G$1" pin="G6"/>
@@
 </segment>
 </net>
-<net name="N$16" class="0">
+<net name="IO7" class="0">
 <segment>
 <pinref part="JP1" gate="A" pin="3"/>
@@
 </segment>
 </net>
-<net name="N$17" class="0">
+<net name="IO10" class="0">
 <segment>
 <pinref part="U$1" gate="G$1" pin="G10"/>
@@
 </segment>
 </net>
-<net name="N$18" class="0">
+<net name="IO4" class="0">
 <segment>
 <pinref part="JP2" gate="A" pin="2"/>
@@
 </segment>
 </net>
-<net name="N$19" class="0">
+<net name="IO3" class="0">
 <segment>
 <pinref part="JP2" gate="A" pin="3"/>
@@
 </segment>
 </net>
-<net name="N$20" class="0">
+<net name="IO2" class="0">
 <segment>
 <pinref part="JP2" gate="A" pin="4"/>
@@
 </segment>
 </net>
-<net name="N$21" class="0">
+<net name="IO1" class="0">
 <segment>
 <pinref part="JP2" gate="A" pin="5"/>
@@
 </sheet>
 </sheets>
-<errors>
-</errors>
 </schematic>
 </drawing>
